Commit message: feat: nav2

File: src/g_robot_description/urdf/g_robot.urdf (robot description, URDF)
Before this commit: robot g_robot, 3 links, 2 joints
Links:
- removed link link_chassis
- removed link link_left_wheel
- removed link link_right_wheel
- added link caster_link, mass 5; collision sphere radius=0.05; visual sphere radius=0.05
- added link chassis_link, mass 10; collision box size=0.5 0.5 0.3; visual box size=0.5 0.5 0.3
- added link left_wheel_joint, mass 1; collision cylinder length=0.04 radius=0.125; visual cylinder length=0.04 radius=0.125
- added link right_wheel_link, mass 1; collision cylinder length=0.04 radius=0.125; visual cylinder length=0.04 radius=0.125
Joints:
- removed joint joint_left_wheel
- removed joint joint_right_wheel
- added joint caster_joint: type fixed, parent caster_link, child chassis_link, origin xyz=-0.175 0 0.1 rpy=0 0 0
- added joint left_wheel_joint: type continuous, parent chassis_link, child left_wheel_joint, origin xyz=-0.1 0.2 -0.025 rpy=0 0 0, axis 0 1 0, limit effort=10000 velocity=1000
- added joint right_wheel_joint: type continuous, parent chassis_link, child right_wheel_link, origin xyz=-0.1 -0.2 -0.025 rpy=0 0 0, axis 0 1 0, limit effort=10000 velocity=1000
