Commit message: feat: all working (needs refactoring)

File: src/g_robot/models/g_robot_v2.urdf (robot description, URDF)
Before this commit: robot g_robot, 6 links, 5 joints
Links:
- removed link base_footprint
- removed link gps_link
- removed link imu_link
Joints:
- removed joint base_joint
- removed joint gps_joint
- removed joint imu_joint

Commit message: chore: refactoring + real robot shape (gazebo & rviz)

File: src/g_robot/models/g_robot_v2.urdf (robot description, URDF)
Before this commit: robot g_robot, 3 links, 2 joints
Links:
- link base_link: geometry collision box size=${base_length} ${base_width} ${base_height}; visual mesh filename=package://g_robot/meshes/base.stl
- link front_caster: geometry collision cylinder length=0.025 radius=0.05; visual cylinder length=0.025 radius=0.05
- link lidar_link: mass 0.114 -> 0.190
Joints:
- joint caster_joint: origin xyz=${caster_xoff} 0.0 ${-(base_height/2)} rpy=0 0 0 -> xyz=${caster_xoff} 0.0 ${caster_zoff} rpy=0 0 0
- joint lidar_joint: origin xyz=0.215 0 0.13 rpy=0 0 0 -> xyz=0 0 0.42 rpy=0 0 0
