Commit message: chore: refactoring + removal of unused files

File: src/g_robot/models/robot_model.urdf (robot description, URDF)
Before this commit: robot g_robot, 3 links, 2 joints
Links:
- link base_link: geometry collision mesh filename=package://g_robot/meshes/base.stl; visual box size=${base_length} ${base_height} ${base_width}
