Commit message: feat: beginning doxygen documentation

File: src/ground_robots_models/models/robot_model.urdf (robot description, URDF)
Before this commit: robot ground_robot, 3 links, 2 joints
Links:
- removed link lidar_link
- added link base_laser, mass 0.190; collision cylinder length=0.18 radius=0.0508; visual cylinder length=0.18 radius=0.0508
Joints:
- joint lidar_joint: child lidar_link -> base_laser
